Commit message: ADD: dae meshes

File: uarm_description/urdf/uarm2.urdf.xacro (robot description, xacro)
@@ -11,5 +11,5 @@
     <visual>
       <geometry>
-        <mesh filename="package://ipa325_robot_descriptions/meshes/uarm/base.dae"/>
+        <mesh filename="package://uarm_description/meshes/arm/base.dae"/>
       </geometry>
     </visual>
@@ -25,5 +25,5 @@
     <visual>
       <geometry>
-        <mesh filename="package://ipa325_robot_descriptions/meshes/uarm/link0.dae"/>
+        <mesh filename="package://uarm_description/meshes/arm/link0.dae"/>
       </geometry>
     </visual>
@@ -39,5 +39,5 @@
     <visual>
       <geometry>
-        <mesh filename="package://ipa325_robot_descriptions/meshes/uarm/link1.dae"/>
+        <mesh filename="package://uarm_description/meshes/arm/link1.dae"/>
       </geometry>
     </visual>
@@ -53,5 +53,5 @@
     <visual>
       <geometry>
-        <mesh filename="package://ipa325_robot_descriptions/meshes/uarm/link2.dae"/>
+        <mesh filename="package://uarm_description/meshes/arm/link2.dae"/>
       </geometry>
     </visual>
@@ -78,5 +78,5 @@
     <visual>
       <geometry>
-        <mesh filename="package://ipa325_robot_descriptions/meshes/uarm/link3.dae"/>
+        <mesh filename="package://uarm_description/meshes/arm/link3.dae"/>
       </geometry>
     </visual>
@@ -92,5 +92,5 @@
     <visual>
       <geometry>
-        <mesh filename="package://ipa325_robot_descriptions/meshes/uarm/tool.dae"/>
+        <mesh filename="package://uarm_description/meshes/arm/tool.dae"/>
       </geometry>
     </visual>

Commit message: WIP: description up2date?

File: uarm_description/urdf/uarm2.urdf.xacro (robot description, xacro)
@@ -16,5 +16,5 @@
     </link>
     <joint name="${prefix}joint_0" type="revolute">
-    <origin xyz="0 0 0.03" rpy="0 0 0"/>
+    <origin xyz="0 0 0.03" rpy="0 0 -${M_PI/3}"/>
       <parent link="${prefix}base_link"/>
       <child link="${prefix}link_0"/>
@@ -30,8 +30,8 @@
     </link>
     <joint name="${prefix}joint_1" type="revolute">
-    <origin xyz="0.02 0 0.07" rpy="${-M_PI/2} 0 0"/>
+    <origin xyz="0.02 0 0.07" rpy="${-M_PI/2} ${M_PI/10} 0"/>
       <parent link="${prefix}link_0"/>
       <child link="${prefix}link_1"/>
-      <axis xyz="0 0 1"/>
+      <axis xyz="0 0 -1"/>
       <limit effort="200" velocity="1.9634" lower="-${M_PI}" upper="${M_PI}"/>
     </joint>
@@ -44,8 +44,18 @@
     </link>
     <joint name="${prefix}joint_2" type="revolute">
-    <origin xyz="0.15 0 0" rpy="0 0 0"/>
+    <origin xyz="0.15 0 0" rpy="0 0 ${M_PI/2}"/>
       <parent link="${prefix}link_1"/>
+      <child link="${prefix}virtual_link_x"/>
+      <axis xyz="0 0 1"/>
+      <limit effort="200" velocity="1.9634" lower="-${M_PI}" upper="${M_PI}"/>
+    </joint>
+    <link name="${prefix}virtual_link_x">
+    </link>
+    <joint name="${prefix}mimic_joint_x" type="revolute">
+    <origin xyz="0 0 0" rpy="0 0 ${-5*M_PI/8}"/>
+      <parent link="${prefix}virtual_link_x"/>
       <child link="${prefix}link_2"/>
-      <axis xyz="0 0 1"/>
+      <mimic joint="${prefix}joint_1" multiplier="-1"/>
+      <axis xyz="0 0 -1"/>
       <limit effort="200" velocity="1.9634" lower="-${M_PI}" upper="${M_PI}"/>
     </joint>
@@ -58,9 +68,9 @@
     </link>
     <joint name="${prefix}mimic_joint_1" type="revolute">
-    <origin xyz="0.16 0 0" rpy="0 0 0"/>
+    <origin xyz="0.16 0 0" rpy="0 0 ${M_PI/2}"/>
       <parent link="${prefix}link_2"/>
       <child link="${prefix}virtual_link_2"/>
-      <mimic joint="${prefix}joint_1" multiplier="-1"/>
-      <axis xyz="0 0 1"/>
+      <mimic joint="${prefix}joint_1" multiplier="0"/>
+      <axis xyz="0 0 -1"/>
       <limit effort="200" velocity="1.9634" lower="-${M_PI}" upper="${M_PI}"/>
     </joint>
@@ -68,5 +78,5 @@
     </link>
     <joint name="${prefix}mimic_joint_2" type="revolute">
-    <origin xyz="0 0 0" rpy="0 0 0"/>
+    <origin xyz="0 0 0" rpy="0 0 ${-7*M_PI/15}"/>
       <parent link="${prefix}virtual_link_2"/>
       <child link="${prefix}link_3"/>
@@ -83,5 +93,5 @@
     </link>
     <joint name="${prefix}joint_3" type="revolute">
-    <origin xyz="0.03 0.01 0" rpy="${-M_PI/2} 0 0"/>
+    <origin xyz="0.03 0.01 0" rpy="${-M_PI/2} ${-M_PI/2} 0"/>
       <parent link="${prefix}link_3"/>
       <child link="${prefix}link_4"/>
@@ -108,5 +118,5 @@
   <link name="world"/>
   <xacro:uArm prefix="" parent="world">
-  <origin xyz="0 0 0" rpy="0 0 0" />
+    <origin xyz="0 0 0" rpy="0 0 0" />
   </xacro:uArm>
 </robot>
